Commit message: Added new meshes and controllers, adjusted joint 4 direction

File: lbr_iiwa_description/urdf/lbr_iiwa.urdf.xacro (robot description, xacro)
@@ -10,5 +10,5 @@
   <link name="world"/>
   <!--lbr-->
-  <xacro:lbr_iiwa name="lbr_iiwa" hardware_interface="$(arg prefix)" parent="world">
+  <xacro:lbr_iiwa name="lbr_iiwa" hardware_interface=" " parent="world">
     <origin xyz="0 0 0.0" rpy="0 0 0" />
   </xacro:lbr_iiwa>

File: lbr_iiwa_description/urdf/lbr_iiwa.xacro (robot description, xacro)
@@ -29,5 +29,5 @@
         <origin xyz="0 0 0" rpy="0 0 0"/>
         <geometry>
-          <mesh filename="package://lbr_iiwa_description/meshes/link_0.stl"/>
+          <mesh filename="package://lbr_iiwa_description/meshes/new/iiwa_r820_link_base/iiwa_r820_link_base_hull.stl"/>
         </geometry>
         <material name="Grey"/>
@@ -36,5 +36,5 @@
         <origin xyz="0 0 0" rpy="0 0 0"/>
         <geometry>
-          <mesh filename="package://lbr_iiwa_description/meshes/coarse/link_0.stl"/>
+          <mesh filename="package://lbr_iiwa_description/meshes/new/iiwa_r820_link_base/iiwa_r820_link_base_hull.stl"/>
         </geometry>
         <material name="Grey"/>
@@ -70,12 +70,12 @@
         <origin xyz="0 0 0" rpy="0 0 0"/>
         <geometry>
-          <mesh filename="package://lbr_iiwa_description/meshes/link_1.stl"/>
-        </geometry>
-        <material name="Orange"/>
-      </visual>
-      <collision>
-        <origin xyz="0 0 0" rpy="0 0 0"/>
-        <geometry>
-          <mesh filename="package://lbr_iiwa_description/meshes/coarse/link_1.stl"/>
+          <mesh filename="package://lbr_iiwa_description/meshes/new/iiwa_r820_link_1/iiwa_r820_link_1_hull.stl"/>
+        </geometry>
+        <material name="Orange"/>
+      </visual>
+      <collision>
+        <origin xyz="0 0 0" rpy="0 0 0"/>
+        <geometry>
+          <mesh filename="package://lbr_iiwa_description/meshes/new/iiwa_r820_link_1/iiwa_r820_link_1_collision.stl"/>
         </geometry>
         <material name="Orange"/>
@@ -105,12 +105,12 @@
         <origin xyz="0 0 0" rpy="0 0 0"/>
         <geometry>
-          <mesh filename="package://lbr_iiwa_description/meshes/link_2.stl"/>
-        </geometry>
-        <material name="Orange"/>
-      </visual>
-      <collision>
-        <origin xyz="0 0 0" rpy="0 0 0"/>
-        <geometry>
-          <mesh filename="package://lbr_iiwa_description/meshes/coarse/link_2.stl"/>
+          <mesh filename="package://lbr_iiwa_description/meshes/new/iiwa_r820_link_2/iiwa_r820_link_2_hull.stl"/>
+        </geometry>
+        <material name="Orange"/>
+      </visual>
+      <collision>
+        <origin xyz="0 0 0" rpy="0 0 0"/>
+        <geometry>
+          <mesh filename="package://lbr_iiwa_description/meshes/new/iiwa_r820_link_2/iiwa_r820_link_2_collision.stl"/>
         </geometry>
         <material name="Orange"/>
@@ -140,16 +140,16 @@
         <origin xyz="0 0 0" rpy="0 0 0"/>
         <geometry>
-          <mesh filename="package://lbr_iiwa_description/meshes/link_3.stl"/>
-        </geometry>
-        <material name="Orange"/>
-      </visual>
-      <collision>
-        <origin xyz="0 0 0" rpy="0 0 0"/>
-        <geometry>
-          <mesh filename="package://lbr_iiwa_description/meshes/coarse/link_3.stl"/>
-        </geometry>
-        <material name="Orange"/>
-      </collision>
-    </link>
+          <mesh filename="package://lbr_iiwa_description/meshes/new/iiwa_r820_link_3/iiwa_r820_link_3_hull.stl"/>
+        </geometry>
+        <material name="Orange"/>
+      </visual>
+      <collision>
+        <origin xyz="0 0 0" rpy="0 0 0"/>
+        <geometry>
+          <mesh filename="package://lbr_iiwa_description/meshes/new/iiwa_r820_link_3/iiwa_r820_link_3_collision.stl"/>
+        </geometry>
+        <material name="Orange"/>
+      </collision>
+   </link>
    <!-- joint between link_3 and link_4 -->
     <joint name="${name}_joint_4" type="revolute">
@@ -157,5 +157,5 @@
       <child link="${name}_link_4"/>
       <origin xyz="0 0 0.2155" rpy="0 0 0"/>
-      <axis xyz="0 1 0"/>
+      <axis xyz="0 -1 0"/>
       <limit lower="${-120 * PI / 180}" upper="${120 * PI / 180}"
              effort="${max_effort}" velocity="${max_velocity}" />
@@ -175,12 +175,12 @@
         <origin xyz="0 0 0" rpy="0 0 0"/>
         <geometry>
-          <mesh filename="package://lbr_iiwa_description/meshes/link_4.stl"/>
-        </geometry>
-        <material name="Orange"/>
-      </visual>
-      <collision>
-        <origin xyz="0 0 0" rpy="0 0 0"/>
-        <geometry>
-          <mesh filename="package://lbr_iiwa_description/meshes/coarse/link_4.stl"/>
+          <mesh filename="package://lbr_iiwa_description/meshes/new/iiwa_r820_link_4/iiwa_r820_link_4_hull.stl"/>
+        </geometry>
+        <material name="Orange"/>
+      </visual>
+      <collision>
+        <origin xyz="0 0 0" rpy="0 0 0"/>
+        <geometry>
+          <mesh filename="package://lbr_iiwa_description/meshes/new/iiwa_r820_link_4/iiwa_r820_link_4_collision.stl"/>
         </geometry>
         <material name="Orange"/>
@@ -210,12 +210,12 @@
         <origin xyz="0 0 0" rpy="0 0 0"/>
         <geometry>
-          <mesh filename="package://lbr_iiwa_description/meshes/link_5.stl"/>
-        </geometry>
-        <material name="Orange"/>
-      </visual>
-      <collision>
-        <origin xyz="0 0 0" rpy="0 0 0"/>
-        <geometry>
-          <mesh filename="package://lbr_iiwa_description/meshes/coarse/link_5.stl"/>
+          <mesh filename="package://lbr_iiwa_description/meshes/new/iiwa_r820_link_5/iiwa_r820_link_5_hull.stl"/>
+        </geometry>
+        <material name="Orange"/>
+      </visual>
+      <collision>
+        <origin xyz="0 0 0" rpy="0 0 0"/>
+        <geometry>
+          <mesh filename="package://lbr_iiwa_description/meshes/new/iiwa_r820_link_5/iiwa_r820_link_5_collision.stl"/>
         </geometry>
         <material name="Orange"/>
@@ -226,5 +226,6 @@
       <parent link="${name}_link_5"/>
       <child link="${name}_link_6"/>
-      <origin xyz="0 -0.0607 0.2155" rpy="0 0 0"/>
+      <!--origin xyz="0 -0.0607 0.2155" rpy="0 0 0"/-->
+      <origin xyz="0 0.0 0.2155" rpy="0 0 0"/>
       <axis xyz="0 1 0"/>
       <limit lower="${-120 * PI / 180}" upper="${120 * PI / 180}"
@@ -245,12 +246,12 @@
         <origin xyz="0 0 0" rpy="0 0 0"/>
         <geometry>
-          <mesh filename="package://lbr_iiwa_description/meshes/link_6.stl"/>
-        </geometry>
-        <material name="Orange"/>
-      </visual>
-      <collision>
-        <origin xyz="0 0 0" rpy="0 0 0"/>
-        <geometry>
-          <mesh filename="package://lbr_iiwa_description/meshes/coarse/link_6.stl"/>
+          <mesh filename="package://lbr_iiwa_description/meshes/new/iiwa_r820_link_6/iiwa_r820_link_6_hull.stl"/>
+        </geometry>
+        <material name="Orange"/>
+      </visual>
+      <collision>
+        <origin xyz="0 0 0" rpy="0 0 0"/>
+        <geometry>
+          <mesh filename="package://lbr_iiwa_description/meshes/new/iiwa_r820_link_6/iiwa_r820_link_6_collision.stl"/>
         </geometry>
         <material name="Orange"/>
@@ -261,5 +262,6 @@
       <parent link="${name}_link_6"/>
       <child link="${name}_link_7"/>
-      <origin xyz="0 0.0607 0.0809" rpy="0 0 0"/>
+      <!--origin xyz="0 0.0607 0.0809" rpy="0 0 0"/-->
+      <origin xyz="0 0 0.0809" rpy="0 0 0"/>
       <axis xyz="0 0 1"/>
       <limit lower="${-175 * PI / 180}" upper="${175 * PI / 180}"
@@ -280,5 +282,5 @@
         <origin xyz="0 0 0" rpy="0 0 0"/>
         <geometry>
-          <mesh filename="package://lbr_iiwa_description/meshes/link_7.stl"/>
+          <mesh filename="package://lbr_iiwa_description/meshes/new/iiwa_r820_link_flange/iiwa_r820_link_flange_hull.stl"/>
         </geometry>
         <material name="Grey"/>
@@ -287,5 +289,5 @@
         <origin xyz="0 0 0" rpy="0 0 0"/>
         <geometry>
-          <mesh filename="package://lbr_iiwa_description/meshes/coarse/link_7.stl"/>
+          <mesh filename="package://lbr_iiwa_description/meshes/new/iiwa_r820_link_flange/iiwa_r820_link_flange_collision.stl"/>
         </geometry>
         <material name="Grey"/>
